File: pcb/I2C-Signal.sch (KiCad schematic (older format))
At the start: 11 parts, among them J13 SM04B-SRSS-TB(LF)(SN), J17 SM04B-SRSS-TB(LF)(SN), J7 Conn_01x04_Male, J8 Conn_01x04_Male, U6 PCA9306DCTR

Commit message: reset code
Parts:
- J13, J17: symbol mainPCB-rescue:SM04B-SRSS-TB(LF)(SN)-Connector_own -> Connector_own:SM04B-SRSS-TB(LF)(SN)
Changed lines of the file:
@@
 EESchema Schematic File Version 4
 LIBS:mainPCB-cache
-EELAYER 29 0
+EELAYER 26 0
 EELAYER END
 $Descr A4 11693 8268
@@
 	2550 950  4700 950
 $Comp
-L mainPCB-rescue:SM04B-SRSS-TB(LF)(SN)-Connector_own J13
+L Connector_own:SM04B-SRSS-TB(LF)(SN) J13
 U 1 1 5CC11751
 P 8950 2400
@@
 $EndComp
 $Comp
-L mainPCB-rescue:SM04B-SRSS-TB(LF)(SN)-Connector_own J17
+L Connector_own:SM04B-SRSS-TB(LF)(SN) J17
 U 1 1 5CC131AA
 P 9900 2400

Commit message: chage LED footprint(D2,D5,D9)
Parts:
- J13, J17: symbol Connector_own:SM04B-SRSS-TB(LF)(SN) -> mainPCB-rescue:SM04B-SRSS-TB(LF)(SN)-Connector_own
Changed lines of the file:
@@
 EESchema Schematic File Version 4
 LIBS:mainPCB-cache
-EELAYER 26 0
+EELAYER 29 0
 EELAYER END
 $Descr A4 11693 8268
@@
 	2550 950  4700 950
 $Comp
-L Connector_own:SM04B-SRSS-TB(LF)(SN) J13
+L mainPCB-rescue:SM04B-SRSS-TB(LF)(SN)-Connector_own J13
 U 1 1 5CC11751
 P 8950 2400
@@
 $EndComp
 $Comp
-L Connector_own:SM04B-SRSS-TB(LF)(SN) J17
+L mainPCB-rescue:SM04B-SRSS-TB(LF)(SN)-Connector_own J17
 U 1 1 5CC131AA
 P 9900 2400
