File: pcb/Relais.sch (KiCad schematic (older format))
At the start: 2 parts, among them K2 CP1SA-12V-Z, U10 NUD3124LT1G

Commit message: reset code
Parts:
- K2: symbol mainPCB-rescue:CP1SA-12V-Z-Relay_own -> Relay_own:CP1SA-12V-Z
- U10: symbol mainPCB-rescue:NUD3124LT1G-GateDriver_own -> GateDriver_own:NUD3124LT1G
Changed lines of the file:
@@
 EESchema Schematic File Version 4
 LIBS:mainPCB-cache
-EELAYER 29 0
+EELAYER 26 0
 EELAYER END
 $Descr A4 11693 8268
@@
 $EndDescr
 $Comp
-L mainPCB-rescue:CP1SA-12V-Z-Relay_own K2
+L Relay_own:CP1SA-12V-Z K2
 U 1 1 5CEBBD54
 P 5950 3100
@@
 $EndComp
 $Comp
-L mainPCB-rescue:NUD3124LT1G-GateDriver_own U10
+L GateDriver_own:NUD3124LT1G U10
 U 1 1 5CEBBF42
 P 6350 2400

Commit message: chage LED footprint(D2,D5,D9)
Parts:
- K2: symbol Relay_own:CP1SA-12V-Z -> mainPCB-rescue:CP1SA-12V-Z-Relay_own
- U10: symbol GateDriver_own:NUD3124LT1G -> mainPCB-rescue:NUD3124LT1G-GateDriver_own
Changed lines of the file:
@@
 EESchema Schematic File Version 4
 LIBS:mainPCB-cache
-EELAYER 26 0
+EELAYER 29 0
 EELAYER END
 $Descr A4 11693 8268
@@
 $EndDescr
 $Comp
-L Relay_own:CP1SA-12V-Z K2
+L mainPCB-rescue:CP1SA-12V-Z-Relay_own K2
 U 1 1 5CEBBD54
 P 5950 3100
@@
 $EndComp
 $Comp
-L GateDriver_own:NUD3124LT1G U10
+L mainPCB-rescue:NUD3124LT1G-GateDriver_own U10
 U 1 1 5CEBBF42
 P 6350 2400
