File: pcb/canTransceiver.sch (KiCad schematic (older format))
At the start: 7 parts, among them IC2 ATA6561-GAQW-N, J12 Conn_02x02_Odd_Even, J18 PTSM-Header-Horizontal-2

Commit message: reset code
Parts:
- IC2: symbol mainPCB-rescue:ATA6561-GAQW-N-Interface_CAN_LIN_own -> Interface_CAN_LIN_own:ATA6561-GAQW-N
- J18: symbol mainPCB-rescue:PTSM-Header-Horizontal-2-Connector_own -> Connector_own:PTSM-Header-Horizontal-2
Changed lines of the file:
@@
 EESchema Schematic File Version 4
 LIBS:mainPCB-cache
-EELAYER 29 0
+EELAYER 26 0
 EELAYER END
 $Descr A4 11693 8268
@@
 $EndDescr
 $Comp
-L mainPCB-rescue:ATA6561-GAQW-N-Interface_CAN_LIN_own IC2
+L Interface_CAN_LIN_own:ATA6561-GAQW-N IC2
 U 1 1 5CACB7D0
 P 5550 2300
@@
 	3500 3100 4500 3100
 $Comp
-L mainPCB-rescue:PTSM-Header-Horizontal-2-Connector_own J18
+L Connector_own:PTSM-Header-Horizontal-2 J18
 U 1 1 5CC27296
 P 9850 2300

Commit message: chage LED footprint(D2,D5,D9)
Parts:
- IC2: symbol Interface_CAN_LIN_own:ATA6561-GAQW-N -> mainPCB-rescue:ATA6561-GAQW-N-Interface_CAN_LIN_own
- J18: symbol Connector_own:PTSM-Header-Horizontal-2 -> mainPCB-rescue:PTSM-Header-Horizontal-2-Connector_own
Changed lines of the file:
@@
 EESchema Schematic File Version 4
 LIBS:mainPCB-cache
-EELAYER 26 0
+EELAYER 29 0
 EELAYER END
 $Descr A4 11693 8268
@@
 $EndDescr
 $Comp
-L Interface_CAN_LIN_own:ATA6561-GAQW-N IC2
+L mainPCB-rescue:ATA6561-GAQW-N-Interface_CAN_LIN_own IC2
 U 1 1 5CACB7D0
 P 5550 2300
@@
 	3500 3100 4500 3100
 $Comp
-L Connector_own:PTSM-Header-Horizontal-2 J18
+L mainPCB-rescue:PTSM-Header-Horizontal-2-Connector_own J18
 U 1 1 5CC27296
 P 9850 2300
