File: pcb/mainPCB.kicad_pcb (KiCad board)
At the start: 4 copper layers, 160 x 73.2 mm, 162 parts, among them IC1 FXL6408UMX, IC2 ATA6561-GAQW-N, IC3 ICL3221EIVZ, J1 PTSM-Header-Horizontal-6, J10 Conn_01x08_Female, J11 Conn_01x08_Female, J12 Conn_02x02_Odd_Even, J13 SM04B-SRSS-TB(LF)(SN), J14 USB_B_Micro, J15 RJ45_Amphenol_RJMG1BD3B8K1ANR, J16 DB9_Male_MountingHoles, J17 SM04B-SRSS-TB(LF)(SN), J18 PTSM-Header-Horizontal-2, J2 Conn_01x02_Male, J3 PTSM-Header-Horizontal-7, J4 CCA-Header-Horizontal-4, J5 PTSM-Header-Horizontal-5, J7 Conn_01x04_Male, J8 Conn_01x04_Male, J9 Conn_01x08_Female, K1 CP1SA-12V-Z, K2 CP1SA-12V-Z, Q1 BC817-40,215, Q2 BC817-40,215, SW1 SW_Push, U1 ESP32-WROOM-32, U10 NUD3124LT1G, U11 LAN8720A, U12 LSM9DS1, U2 AZ1117-3.3, U3 VNH7070AS, U4 ADS1115IDGS, U5 VNH7070AS, U6 PCA9306DCTR, U7 TPD3E001DRLR, U8 CP2102N-A01-GQFN24, U9 VNH7070AS

Commit message: change LED footprint
Parts:
- D2, D5, D9: footprint Capacitor_SMD:C_0805_2012Metric -> LED_SMD:LED_0805_2012Metric
Other:
- rule via_min_size: 0.4 -> 0.6

Commit message: F.Fab arrangement
Parts:
- C35: value 100n/16V -> 100n
- D2: value LED/blue -> LED/yellow
- IC2: value ATA6561-GAQW-N -> ATA6561
Other:
- board text added: "ESP-F9P-IO-Board Version 2.1m"
- board text added: "F9P"
- board text added: "POWER"
- board text removed: "ESP-F9P-IO-Board Version 2.1"
