File: pcb/mainPCB.kicad_pcb (KiCad board)
At the start: 4 copper layers, 160 x 73.2 mm, 162 parts, among them IC1 FXL6408UMX, IC2 ATA6561, IC3 ICL3221EIVZ, J1 PTSM-Header-Horizontal-6, J10 Conn_01x08_Female, J11 Conn_01x08_Female, J12 Conn_02x02_Odd_Even, J13 SM04B-SRSS-TB(LF)(SN), J14 USB_B_Micro, J15 RJ45_Amphenol_RJMG1BD3B8K1ANR, J16 DB9_Male_MountingHoles, J17 SM04B-SRSS-TB(LF)(SN), J18 PTSM-Header-Horizontal-2, J2 Conn_01x02_Male, J3 PTSM-Header-Horizontal-7, J4 CCA-Header-Horizontal-4, J5 PTSM-Header-Horizontal-5, J7 Conn_01x04_Male, J8 Conn_01x04_Male, J9 Conn_01x08_Female, K1 CP1SA-12V-Z, K2 CP1SA-12V-Z, Q1 BC817-40,215, Q2 BC817-40,215, SW1 SW_Push, U1 ESP32-WROOM-32, U10 NUD3124LT1G, U11 LAN8720A, U12 LSM9DS1, U2 AZ1117-3.3, U3 VNH7070AS, U4 ADS1115IDGS, U5 VNH7070AS, U6 PCA9306DCTR, U7 TPD3E001DRLR, U8 CP2102N-A01-GQFN24, U9 VNH7070AS

Commit message: reset code
Parts:
- removed L1: 22u, Inductor_SMD:L_0805_2012Metric
- removed REF** (x4): Fiducial_1mm_Dia_2mm_Outer, Fiducial:Fiducial_1mm_Dia_2mm_Outer
- added R2: 24, Resistor_SMD:R_0805_2012Metric, F.Cu at (132.7, 51.6)
- added REF*1: Fiducial, Fiducial:Fiducial_1mm_Dia_2mm_Outer, F.Cu at (19.7, 39.7)
- added REF*2: Fiducial, Fiducial:Fiducial_1mm_Dia_2mm_Outer, F.Cu at (175.1, 39.7)
- added REF*3: Fiducial, Fiducial:Fiducial_1mm_Dia_2mm_Outer, F.Cu at (19.2, 108.7)
- added REF*4: Fiducial, Fiducial:Fiducial_1mm_Dia_2mm_Outer, F.Cu at (175.4, 108.7)
- C10: value 10u -> 22u
- C35: value 100n -> 100n/16V
- D2: value LED/yellow -> LED/blue; footprint LED_SMD:LED_0805_2012Metric -> Capacitor_SMD:C_0805_2012Metric
- D5, D9: footprint LED_SMD:LED_0805_2012Metric -> Capacitor_SMD:C_0805_2012Metric
- IC2: value ATA6561 -> ATA6561-GAQW-N
- moved C46 1.49 mm to (157.8, 100.7), turned to 0 degrees
Connections:
- IC3 pad 12: GND -> +3V3
Routing:
- net +3V3: track 81.6 -> 87.7 mm
- net GND: track 288.0 -> 290.5 mm
- net Net-(C23-Pad1): track 5.37 -> 7.43 mm
Other:
- rule via_min_size: 0.6 -> 0.4
- board text added: "ESP-F9P-IO-Board Version 2.2"
- board text removed: "ESP-F9P-IO-Board Version 2.1m"
- board text removed: "F9P"
- board text removed: "POWER"
