File: pcb/ADS-Input.sch (KiCad schematic (older format))
At the start: 12 parts, among them J5 PTSM-Header-Horizontal-5, U4 ADS1115IDGS

Commit message: chage LED footprint(D2,D5,D9)
Parts:
- J5: symbol Connector_own:PTSM-Header-Horizontal-5 -> mainPCB-rescue:PTSM-Header-Horizontal-5-Connector_own
Changed lines of the file:
@@
 EESchema Schematic File Version 4
 LIBS:mainPCB-cache
-EELAYER 26 0
+EELAYER 29 0
 EELAYER END
 $Descr A4 11693 8268
@@
 	4900 3200 6000 3200
 $Comp
-L Connector_own:PTSM-Header-Horizontal-5 J5
+L mainPCB-rescue:PTSM-Header-Horizontal-5-Connector_own J5
 U 1 1 5CCCDB32
 P 1250 3300

Commit message: reset code
Parts:
- J5: symbol mainPCB-rescue:PTSM-Header-Horizontal-5-Connector_own -> Connector_own:PTSM-Header-Horizontal-5
- R2: renamed from L1; value 22u -> 24; footprint Inductor_SMD:L_0805_2012Metric -> Resistor_SMD:R_0805_2012Metric; symbol Device:L -> Device:R
Changed lines of the file:
@@
 EESchema Schematic File Version 4
 LIBS:mainPCB-cache
-EELAYER 29 0
+EELAYER 26 0
 EELAYER END
 $Descr A4 11693 8268
@@
 Connection ~ 7550 2350
 $Comp
-L Device:L L1
+L Device:R R2
 U 1 1 5CA41C10
 P 8800 2050
-F 0 "L1" V 8990 2050 50  0000 C CNN
-F 1 "22u" V 8899 2050 50  0000 C CNN
-F 2 "Inductor_SMD:L_0805_2012Metric" H 8800 2050 50  0001 C CNN
+F 0 "R2" V 8990 2050 50  0000 C CNN
+F 1 "24" V 8899 2050 50  0000 C CNN
+F 2 "Resistor_SMD:R_0805_2012Metric" H 8800 2050 50  0001 C CNN
 F 3 "~" H 8800 2050 50  0001 C CNN
 	1    8800 2050
@@
 	4900 3200 6000 3200
 $Comp
-L mainPCB-rescue:PTSM-Header-Horizontal-5-Connector_own J5
+L Connector_own:PTSM-Header-Horizontal-5 J5
 U 1 1 5CCCDB32
 P 1250 3300
