File: pcb/RS232.sch (KiCad schematic (older format))
At the start: 7 parts, among them IC3 ICL3221EIVZ, J16 DB9_Male_MountingHoles

Commit message: chage LED footprint(D2,D5,D9)
Parts:
- IC3: symbol Interface_UART_own:ICL3221EIVZ -> mainPCB-rescue:ICL3221EIVZ-Interface_UART_own
Changed lines of the file:
@@
 EESchema Schematic File Version 4
 LIBS:mainPCB-cache
-EELAYER 26 0
+EELAYER 29 0
 EELAYER END
 $Descr A4 11693 8268
@@
 $EndDescr
 $Comp
-L Interface_UART_own:ICL3221EIVZ IC3
+L mainPCB-rescue:ICL3221EIVZ-Interface_UART_own IC3
 U 1 1 5CF77802
 P 5600 3150

Commit message: reset code
Parts:
- IC3: symbol mainPCB-rescue:ICL3221EIVZ-Interface_UART_own -> Interface_UART_own:ICL3221EIVZ
Connections:
- net +3V3: now also IC3.12 (FORCEON)
- net GND: no longer IC3.12 (FORCEON)
Changed lines of the file:
@@
 EESchema Schematic File Version 4
 LIBS:mainPCB-cache
-EELAYER 29 0
+EELAYER 26 0
 EELAYER END
 $Descr A4 11693 8268
@@
 $EndDescr
 $Comp
-L mainPCB-rescue:ICL3221EIVZ-Interface_UART_own IC3
+L Interface_UART_own:ICL3221EIVZ IC3
 U 1 1 5CF77802
 P 5600 3150
@@
 Wire Wire Line
 	7100 1750 6400 1750
-Wire Wire Line
-	6250 3200 7100 3200
-Wire Wire Line
-	7100 3200 7100 3000
-Connection ~ 7100 3000
 Text HLabel 6250 3300 2    50   BiDi ~ 0
 UART_TX
@@
 Wire Wire Line
 	8100 1750 7550 1750
+Wire Wire Line
+	6400 2900 6400 3200
+Wire Wire Line
+	6400 3200 6250 3200
 $EndSCHEMATC
