File: pcb/mainPCB.sch (KiCad schematic (older format))
At the start: 31 parts, among them IC1 FXL6408UMX, J1 PTSM-Header-Horizontal-6, J2 Conn_01x02_Male, J3 PTSM-Header-Horizontal-7, J4 CCA-Header-Horizontal-4, SW1 SW_Push, U1 ESP32-WROOM-32

Commit message: chage LED footprint(D2,D5,D9)
Parts:
- D2: value LED/blue -> LED/yellow; footprint Capacitor_SMD:C_0805_2012Metric -> LED_SMD:LED_0805_2012Metric
- IC1: symbol Interface_Expansion_own:FXL6408UMX -> mainPCB-rescue:FXL6408UMX-Interface_Expansion_own
- J1: symbol Connector_own:PTSM-Header-Horizontal-6 -> mainPCB-rescue:PTSM-Header-Horizontal-6-Connector_own
- J3: symbol Connector_own:PTSM-Header-Horizontal-7 -> mainPCB-rescue:PTSM-Header-Horizontal-7-Connector_own
- J4: symbol Connector_own:CCA-Header-Horizontal-4 -> mainPCB-rescue:CCA-Header-Horizontal-4-Connector_own
Changed lines of the file:
@@
 EESchema Schematic File Version 4
 LIBS:mainPCB-cache
-EELAYER 26 0
+EELAYER 29 0
 EELAYER END
 $Descr A4 11693 8268
@@
 Connection ~ 2550 2400
 $Comp
-L Interface_Expansion_own:FXL6408UMX IC1
+L mainPCB-rescue:FXL6408UMX-Interface_Expansion_own IC1
 U 1 1 5CE85D35
 P 4000 4950
@@
 P 5000 6650
 F 0 "D2" H 4992 6395 50  0000 C CNN
-F 1 "LED/blue" H 4992 6486 50  0000 C CNN
-F 2 "Capacitor_SMD:C_0805_2012Metric" H 5000 6650 50  0001 C CNN
+F 1 "LED/yellow" H 4992 6486 50  0000 C CNN
+F 2 "LED_SMD:LED_0805_2012Metric" H 5000 6650 50  0001 C CNN
 F 3 "~" H 5000 6650 50  0001 C CNN
 	1    5000 6650
@@
 	7000 2400 7000 3000
 $Comp
-L Connector_own:PTSM-Header-Horizontal-7 J3
+L mainPCB-rescue:PTSM-Header-Horizontal-7-Connector_own J3
 U 1 1 5CC33CA3
 P 7800 4950
@@
 	5000 2400 3600 2400
 $Comp
-L Connector_own:PTSM-Header-Horizontal-6 J1
+L mainPCB-rescue:PTSM-Header-Horizontal-6-Connector_own J1
 U 1 1 5CD05128
 P 1250 1650
@@
 	8300 4800 8200 4800
 $Comp
-L Connector_own:CCA-Header-Horizontal-4 J4
+L mainPCB-rescue:CCA-Header-Horizontal-4-Connector_own J4
 U 1 1 5CE0099D
 P 10900 4550

Commit message: reset code
Parts:
- added REF*1, REF*2, REF*3, REF*4: Fiducial, Fiducial:Fiducial_1mm_Dia_2mm_Outer, symbol Virtual_own:Fiducial
- D2: value LED/yellow -> LED/blue; footprint LED_SMD:LED_0805_2012Metric -> Capacitor_SMD:C_0805_2012Metric
- IC1: symbol mainPCB-rescue:FXL6408UMX-Interface_Expansion_own -> Interface_Expansion_own:FXL6408UMX
- J1: symbol mainPCB-rescue:PTSM-Header-Horizontal-6-Connector_own -> Connector_own:PTSM-Header-Horizontal-6
- J3: symbol mainPCB-rescue:PTSM-Header-Horizontal-7-Connector_own -> Connector_own:PTSM-Header-Horizontal-7
- J4: symbol mainPCB-rescue:CCA-Header-Horizontal-4-Connector_own -> Connector_own:CCA-Header-Horizontal-4
Changed lines of the file:
@@
 EESchema Schematic File Version 4
 LIBS:mainPCB-cache
-EELAYER 29 0
+EELAYER 26 0
 EELAYER END
 $Descr A4 11693 8268
@@
 Connection ~ 2550 2400
 $Comp
-L mainPCB-rescue:FXL6408UMX-Interface_Expansion_own IC1
+L Interface_Expansion_own:FXL6408UMX IC1
 U 1 1 5CE85D35
 P 4000 4950
@@
 P 5000 6650
 F 0 "D2" H 4992 6395 50  0000 C CNN
-F 1 "LED/yellow" H 4992 6486 50  0000 C CNN
-F 2 "LED_SMD:LED_0805_2012Metric" H 5000 6650 50  0001 C CNN
+F 1 "LED/blue" H 4992 6486 50  0000 C CNN
+F 2 "Capacitor_SMD:C_0805_2012Metric" H 5000 6650 50  0001 C CNN
 F 3 "~" H 5000 6650 50  0001 C CNN
 	1    5000 6650
@@
 	7000 2400 7000 3000
 $Comp
-L mainPCB-rescue:PTSM-Header-Horizontal-7-Connector_own J3
+L Connector_own:PTSM-Header-Horizontal-7 J3
 U 1 1 5CC33CA3
 P 7800 4950
@@
 	5000 2400 3600 2400
 $Comp
-L mainPCB-rescue:PTSM-Header-Horizontal-6-Connector_own J1
+L Connector_own:PTSM-Header-Horizontal-6 J1
 U 1 1 5CD05128
 P 1250 1650
@@
 	8300 4800 8200 4800
 $Comp
-L mainPCB-rescue:CCA-Header-Horizontal-4-Connector_own J4
+L Connector_own:CCA-Header-Horizontal-4 J4
 U 1 1 5CE0099D
 P 10900 4550
@@
 Wire Wire Line
 	2800 4800 2800 5550
+$Comp
+L Virtual_own:Fiducial REF*4
+U 1 1 5D4DF8B0
+P 1600 7650
+F 0 "REF*4" H 1555 7700 50  0000 L CNN
+F 1 "Fiducial" H 1600 7700 50  0001 C CNN
+F 2 "Fiducial:Fiducial_1mm_Dia_2mm_Outer" H 1600 7650 50  0001 C CNN
+F 3 "" H 1600 7650 50  0001 C CNN
+	1    1600 7650
+	1    0    0    -1
+$EndComp
+$Comp
+L Virtual_own:Fiducial REF*3
+U 1 1 5D4DF928
+P 1600 7500
+F 0 "REF*3" H 1555 7550 50  0000 L CNN
+F 1 "Fiducial" H 1600 7550 50  0001 C CNN
+F 2 "Fiducial:Fiducial_1mm_Dia_2mm_Outer" H 1600 7500 50  0001 C CNN
+F 3 "" H 1600 7500 50  0001 C CNN
+	1    1600 7500
+	1    0    0    -1
+$EndComp
+$Comp
+L Virtual_own:Fiducial REF*2
+U 1 1 5D4DF980
+P 1600 7350
+F 0 "REF*2" H 1555 7400 50  0000 L CNN
+F 1 "Fiducial" H 1600 7400 50  0001 C CNN
+F 2 "Fiducial:Fiducial_1mm_Dia_2mm_Outer" H 1600 7350 50  0001 C CNN
+F 3 "" H 1600 7350 50  0001 C CNN
+	1    1600 7350
+	1    0    0    -1
+$EndComp
+$Comp
+L Virtual_own:Fiducial REF*1
+U 1 1 5D4DF9D6
+P 1600 7200
+F 0 "REF*1" H 1555 7250 50  0000 L CNN
+F 1 "Fiducial" H 1600 7250 50  0001 C CNN
+F 2 "Fiducial:Fiducial_1mm_Dia_2mm_Outer" H 1600 7200 50  0001 C CNN
+F 3 "" H 1600 7200 50  0001 C CNN
+	1    1600 7200
+	1    0    0    -1
+$EndComp
 $EndSCHEMATC
