File: pcb/motorDriver.sch (KiCad schematic (older format))
At the start: 3 parts, among them U3 VNH7070AS

Commit message: chage LED footprint(D2,D5,D9)
Parts:
- U3: symbol Driver_Motor_own:VNH7070AS -> mainPCB-rescue:VNH7070AS-Driver_Motor_own
Changed lines of the file:
@@
 EESchema Schematic File Version 4
 LIBS:mainPCB-cache
-EELAYER 26 0
+EELAYER 29 0
 EELAYER END
 $Descr A4 11693 8268
@@
 PWM
 $Comp
-L Driver_Motor_own:VNH7070AS U3
+L mainPCB-rescue:VNH7070AS-Driver_Motor_own U3
 U 1 1 5C445805
 P 3300 1350

Commit message: reset code
Parts:
- U3: symbol mainPCB-rescue:VNH7070AS-Driver_Motor_own -> Driver_Motor_own:VNH7070AS
Changed lines of the file:
@@
 EESchema Schematic File Version 4
 LIBS:mainPCB-cache
-EELAYER 29 0
+EELAYER 26 0
 EELAYER END
 $Descr A4 11693 8268
@@
 PWM
 $Comp
-L mainPCB-rescue:VNH7070AS-Driver_Motor_own U3
+L Driver_Motor_own:VNH7070AS U3
 U 1 1 5C445805
 P 3300 1350
