File: pcb/powerSupply.sch (KiCad schematic (older format))
At the start: 18 parts, among them K1 CP1SA-12V-Z, U2 AZ1117-3.3

Commit message: chage LED footprint(D2,D5,D9)
Parts:
- D5: footprint Capacitor_SMD:C_0805_2012Metric -> LED_SMD:LED_0805_2012Metric_Castellated
- D9: footprint Capacitor_SMD:C_0805_2012Metric -> LED_SMD:LED_0805_2012Metric
- K1: symbol Relay_own:CP1SA-12V-Z -> mainPCB-rescue:CP1SA-12V-Z-Relay_own
- PS1: symbol Regulator_Switching_own:V78E05-1000-SMT-TR -> mainPCB-rescue:V78E05-1000-SMT-TR-Regulator_Switching_own
Changed lines of the file:
@@
 EESchema Schematic File Version 4
 LIBS:mainPCB-cache
-EELAYER 26 0
+EELAYER 29 0
 EELAYER END
 $Descr A4 11693 8268
@@
 F 0 "D5" V 1838 1483 50  0000 R CNN
 F 1 "LED/red" V 1747 1483 50  0000 R CNN
-F 2 "Capacitor_SMD:C_0805_2012Metric" H 1800 1600 50  0001 C CNN
+F 2 "LED_SMD:LED_0805_2012Metric_Castellated" H 1800 1600 50  0001 C CNN
 F 3 "~" H 1800 1600 50  0001 C CNN
 	1    1800 1600
@@
 F 0 "D9" V 10238 3733 50  0000 R CNN
 F 1 "LED/green" V 10147 3733 50  0000 R CNN
-F 2 "Capacitor_SMD:C_0805_2012Metric" H 10200 3850 50  0001 C CNN
+F 2 "LED_SMD:LED_0805_2012Metric" H 10200 3850 50  0001 C CNN
 F 3 "~" H 10200 3850 50  0001 C CNN
 	1    10200 3850
@@
 	1800 1450 1800 1000
 $Comp
-L Regulator_Switching_own:V78E05-1000-SMT-TR PS1
+L mainPCB-rescue:V78E05-1000-SMT-TR-Regulator_Switching_own PS1
 U 1 1 5C999BE8
 P 7500 1700
@@
 	8400 2000 8400 4650
 $Comp
-L Relay_own:CP1SA-12V-Z K1
+L mainPCB-rescue:CP1SA-12V-Z-Relay_own K1
 U 1 1 5CB977B6
 P 2850 2200

Commit message: reset code
Parts:
- C10: value 10u -> 22u
- D5: footprint LED_SMD:LED_0805_2012Metric_Castellated -> Capacitor_SMD:C_0805_2012Metric
- D9: footprint LED_SMD:LED_0805_2012Metric -> Capacitor_SMD:C_0805_2012Metric
- K1: symbol mainPCB-rescue:CP1SA-12V-Z-Relay_own -> Relay_own:CP1SA-12V-Z
- PS1: symbol mainPCB-rescue:V78E05-1000-SMT-TR-Regulator_Switching_own -> Regulator_Switching_own:V78E05-1000-SMT-TR
Changed lines of the file:
@@
 EESchema Schematic File Version 4
 LIBS:mainPCB-cache
-EELAYER 29 0
+EELAYER 26 0
 EELAYER END
 $Descr A4 11693 8268
@@
 P 9150 3200
 F 0 "C10" H 9265 3246 50  0000 L CNN
-F 1 "10u" H 9265 3155 50  0000 L CNN
+F 1 "22u" H 9265 3155 50  0000 L CNN
 F 2 "Capacitor_SMD:C_0805_2012Metric" H 9188 3050 50  0001 C CNN
 F 3 "~" H 9150 3200 50  0001 C CNN
@@
 F 0 "D5" V 1838 1483 50  0000 R CNN
 F 1 "LED/red" V 1747 1483 50  0000 R CNN
-F 2 "LED_SMD:LED_0805_2012Metric_Castellated" H 1800 1600 50  0001 C CNN
+F 2 "Capacitor_SMD:C_0805_2012Metric" H 1800 1600 50  0001 C CNN
 F 3 "~" H 1800 1600 50  0001 C CNN
 	1    1800 1600
@@
 F 0 "D9" V 10238 3733 50  0000 R CNN
 F 1 "LED/green" V 10147 3733 50  0000 R CNN
-F 2 "LED_SMD:LED_0805_2012Metric" H 10200 3850 50  0001 C CNN
+F 2 "Capacitor_SMD:C_0805_2012Metric" H 10200 3850 50  0001 C CNN
 F 3 "~" H 10200 3850 50  0001 C CNN
 	1    10200 3850
@@
 	1800 1450 1800 1000
 $Comp
-L mainPCB-rescue:V78E05-1000-SMT-TR-Regulator_Switching_own PS1
+L Regulator_Switching_own:V78E05-1000-SMT-TR PS1
 U 1 1 5C999BE8
 P 7500 1700
@@
 	8400 2000 8400 4650
 $Comp
-L mainPCB-rescue:CP1SA-12V-Z-Relay_own K1
+L Relay_own:CP1SA-12V-Z K1
 U 1 1 5CB977B6
 P 2850 2200
