File: pcb/usbUart.sch (KiCad schematic (older format))
At the start: 19 parts, among them J14 USB_B_Micro, Q1 BC817-40,215, Q2 BC817-40,215, U7 TPD3E001DRLR, U8 CP2102N-A01-GQFN24

Commit message: chage LED footprint(D2,D5,D9)
Parts:
- Q1, Q2: symbol Transistor_BJT_own:BC817-40,215 -> mainPCB-rescue:BC817-40,215-Transistor_BJT_own
Changed lines of the file:
@@
 EESchema Schematic File Version 4
 LIBS:mainPCB-cache
-EELAYER 26 0
+EELAYER 29 0
 EELAYER END
 $Descr A4 11693 8268
@@
 	10100 5200 10250 5200
 $Comp
-L Transistor_BJT_own:BC817-40,215 Q2
+L mainPCB-rescue:BC817-40,215-Transistor_BJT_own Q2
 U 1 1 5CB02B3A
 P 9750 3650
@@
 $EndComp
 $Comp
-L Transistor_BJT_own:BC817-40,215 Q1
+L mainPCB-rescue:BC817-40,215-Transistor_BJT_own Q1
 U 1 1 5CB02C43
 P 8650 4900

Commit message: reset code
Parts:
- Q1, Q2: symbol mainPCB-rescue:BC817-40,215-Transistor_BJT_own -> Transistor_BJT_own:BC817-40,215
Changed lines of the file:
@@
 EESchema Schematic File Version 4
 LIBS:mainPCB-cache
-EELAYER 29 0
+EELAYER 26 0
 EELAYER END
 $Descr A4 11693 8268
@@
 	10100 5200 10250 5200
 $Comp
-L mainPCB-rescue:BC817-40,215-Transistor_BJT_own Q2
+L Transistor_BJT_own:BC817-40,215 Q2
 U 1 1 5CB02B3A
 P 9750 3650
@@
 $EndComp
 $Comp
-L mainPCB-rescue:BC817-40,215-Transistor_BJT_own Q1
+L Transistor_BJT_own:BC817-40,215 Q1
 U 1 1 5CB02C43
 P 8650 4900
